Commit message: Fix wheel separation from measured 177mm; tighten SLAM scan matcher
Corrects wheel_separation in diff_drive_controller (0.17→0.177m) and
URDF joint origins (±0.07→±0.0885m) to match physically measured axle
width. Also raises link_match_minimum_response_fine (0.1→0.35) to
reject poor scan matches that caused duplicate walls during mapping.

Co-Authored-By: Claude Sonnet 4.6 <noreply@anthropic.com>

File: src/bumperbot_description/urdf/bumperbot.urdf.xacro (robot description, xacro)
@@ -59,5 +59,5 @@
         <child link="wheel_right_link" />
         <axis xyz="0 1 0" />
-        <origin rpy="0 0 0" xyz="0 -0.07 0" />
+        <origin rpy="0 0 0" xyz="0 -0.0885 0" />
     </joint>
     <link name="wheel_left_link">
@@ -85,5 +85,5 @@
         <child link="wheel_left_link" />
         <axis xyz="0 1 0" />
-        <origin rpy="0 0 0" xyz="0 0.07 0" />
+        <origin rpy="0 0 0" xyz="0 0.0885 0" />
     </joint>
     <link name="caster_front_link">

Commit message: Fix laser_joint 180-degree yaw mismatch with base_link/odom/map frames
laser_link's TF was rotated 180 degrees relative to base_link, odom, and map,
which corrupted SLAM's scan matching against the consistent wheel-odometry
heading and caused map duplication when driving straight. Remove the
erroneous yaw offset.

Co-Authored-By: Claude Sonnet 4.6 <noreply@anthropic.com>

File: src/bumperbot_description/urdf/bumperbot.urdf.xacro (robot description, xacro)
@@ -187,5 +187,5 @@
     </link>
     <joint name="laser_joint" type="fixed">
-        <origin xyz="0 0 0.1208" rpy="0 0 3.14" />
+        <origin xyz="0 0 0.1208" rpy="0 0 0" />
         <parent link="base_link" />
         <child link="laser_link" />
